File: 1. PSU/PCB/PSU KiCad Project/zasilacz v2.kicad_pcb (KiCad board)
At the start: 2 copper layers, 47 x 51 mm, 23 parts, among them J1 USB_B, J2 Conn_01x04, J3 Conn_01x04, J4 Conn_01x04, J5 Conn_01x04, J6 Conn_01x04, U1 MIC4576, U2 TC7660H

Commit message: PSU layout
Routing:
- net GND: track 225.6 -> 221.1 mm, vias 2 -> 0
Changed lines of the file:
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@@
     (thickness 1.6)
     (drawings 5)
-    (tracks 148)
+    (tracks 145)
     (zones 0)
     (modules 23)
@@
   )
   (setup
-    (last_trace_width 0.8)
+    (last_trace_width 0.25)
     (user_trace_width 0.6)
     (user_trace_width 0.8)
@@
   (segment (start 152.5 84) (end 148 84) (width 0.8) (layer B.Cu) (net 3) (status 10))
   (segment (start 167.5 85.5) (end 168 85.5) (width 0.8) (layer B.Cu) (net 4))
-  (via (at 163.5 85.5) (size 1.6) (drill 0.8) (layers F.Cu B.Cu) (net 4))
-  (segment (start 168 85.5) (end 163.5 85.5) (width 0.8) (layer F.Cu) (net 4))
-  (via (at 168 85.5) (size 1.6) (drill 0.8) (layers F.Cu B.Cu) (net 4))
   (segment (start 134.5 78) (end 135 78) (width 0.8) (layer B.Cu) (net 4) (status 10))
   (segment (start 134.5 71) (end 135 71) (width 0.8) (layer B.Cu) (net 4) (status 10))

Commit message: Amiga rulez
Parts:
- moved J4 85.8 mm to (62.7, 55.0)
- moved C1 85.8 mm to (75.8, 50.0)
- moved C2 85.8 mm to (58.8, 42.0)
- moved C3 85.8 mm to (58.8, 49.0)
- moved C4 85.8 mm to (74.8, 63.0)
- moved C5 85.8 mm to (73.3, 36.0)
- moved C6 85.8 mm to (46.3, 52.5)
- moved C7 85.8 mm to (49.3, 52.5)
- moved D1 85.8 mm to (85.3, 28.0)
- moved J1 85.8 mm to (56.3, 34.0)
- moved J2 85.8 mm to (52.5, 55.0)
- moved J3 85.8 mm to (57.5, 55.0)
- moved J5 85.8 mm to (67.3, 55.0)
- moved J6 85.8 mm to (71.8, 55.0)
- moved L1 85.8 mm to (81.8, 33.0)
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