File: 1. PSU/PCB/PSU KiCad Project/zasilacz v2.sch (KiCad schematic (older format))
At the start: 19 parts, among them J1 USB_B, J2 Conn_01x04, J3 Conn_01x04, J4 Conn_01x04, J5 Conn_01x04, J6 Conn_01x04, U1 MIC4576, U2 TC7660H

Commit message: nowe rzeczy
Parts:
- C1, C4: value C -> 1u
- C2: value CP -> 470u
- C3, C6, C7: value C -> 100n
- C5: value CP -> 1000u
- L1: value L -> 33u
- R1: value R -> 2k5
- R2: value R -> 1k5
Changed lines of the file:
@@
 LIBS:contrib
 LIBS:valves
-LIBS:Różne biblioteki Artura
 LIBS:zasilacz v2-cache
 EELAYER 25 0
@@
 P 2200 2650
 F 0 "L1" V 2150 2650 50  0000 C CNN
-F 1 "L" V 2275 2650 50  0000 C CNN
+F 1 "33u" V 2275 2650 50  0000 C CNN
 F 2 "Inductors_THT:L_Radial_D8.7mm_P5.00mm_Fastron_07HCP" H 2200 2650 50  0001 C CNN
 F 3 "" H 2200 2650 50  0001 C CNN
@@
 P 2450 2950
 F 0 "C5" H 2475 3050 50  0000 L CNN
-F 1 "CP" H 2475 2850 50  0000 L CNN
+F 1 "1000u" H 2475 2850 50  0000 L CNN
 F 2 "Capacitors_THT:CP_Radial_D10.0mm_P5.00mm" H 2488 2800 50  0001 C CNN
 F 3 "" H 2450 2950 50  0001 C CNN
@@
 P 2750 2950
 F 0 "R1" V 2830 2950 50  0000 C CNN
-F 1 "R" V 2750 2950 50  0000 C CNN
+F 1 "2k5" V 2750 2950 50  0000 C CNN
 F 2 "Resistors_THT:R_Axial_DIN0204_L3.6mm_D1.6mm_P7.62mm_Horizontal" V 2680 2950 50  0001 C CNN
 F 3 "" H 2750 2950 50  0001 C CNN
@@
 P 3000 2950
 F 0 "R2" V 3080 2950 50  0000 C CNN
-F 1 "R" V 3000 2950 50  0000 C CNN
+F 1 "1k5" V 3000 2950 50  0000 C CNN
 F 2 "Resistors_THT:R_Axial_DIN0204_L3.6mm_D1.6mm_P7.62mm_Horizontal" V 2930 2950 50  0001 C CNN
 F 3 "" H 3000 2950 50  0001 C CNN
@@
 P 1700 4850
 F 0 "C1" H 1725 4950 50  0000 L CNN
-F 1 "C" H 1725 4750 50  0000 L CNN
+F 1 "1u" H 1725 4750 50  0000 L CNN
 F 2 "Capacitors_THT:C_Disc_D4.3mm_W1.9mm_P5.00mm" H 1738 4700 50  0001 C CNN
 F 3 "" H 1700 4850 50  0001 C CNN
@@
 P 2300 4200
 F 0 "C4" H 2325 4300 50  0000 L CNN
-F 1 "C" H 2325 4100 50  0000 L CNN
+F 1 "1u" H 2325 4100 50  0000 L CNN
 F 2 "Capacitors_THT:C_Disc_D4.3mm_W1.9mm_P5.00mm" H 2338 4050 50  0001 C CNN
 F 3 "" H 2300 4200 50  0001 C CNN
@@
 P 1900 1450
 F 0 "C2" H 1925 1550 50  0000 L CNN
-F 1 "CP" H 1925 1350 50  0000 L CNN
+F 1 "470u" H 1925 1350 50  0000 L CNN
 F 2 "Capacitors_THT:CP_Radial_D10.0mm_P5.00mm" H 1938 1300 50  0001 C CNN
 F 3 "" H 1900 1450 50  0001 C CNN
@@
 P 2200 1450
 F 0 "C3" H 2225 1550 50  0000 L CNN
-F 1 "C" H 2225 1350 50  0000 L CNN
+F 1 "100n" H 2225 1350 50  0000 L CNN
 F 2 "Capacitors_THT:C_Disc_D4.3mm_W1.9mm_P5.00mm" H 2238 1300 50  0001 C CNN
 F 3 "" H 2200 1450 50  0001 C CNN
@@
 P 2500 4950
 F 0 "C6" H 2525 5050 50  0000 L CNN
-F 1 "C" H 2525 4850 50  0000 L CNN
+F 1 "100n" H 2525 4850 50  0000 L CNN
 F 2 "Capacitors_THT:C_Disc_D4.3mm_W1.9mm_P5.00mm" H 2538 4800 50  0001 C CNN
 F 3 "" H 2500 4950 50  0001 C CNN
@@
 P 2750 4950
 F 0 "C7" H 2775 5050 50  0000 L CNN
-F 1 "C" H 2775 4850 50  0000 L CNN
+F 1 "100n" H 2775 4850 50  0000 L CNN
 F 2 "Capacitors_THT:C_Disc_D4.3mm_W1.9mm_P5.00mm" H 2788 4800 50  0001 C CNN
 F 3 "" H 2750 4950 50  0001 C CNN

Commit message: Amiga rulez
Parts:
- C1, C3, C4, C6, C7: symbol C -> zasilacz-v2-rescue:C
- C2, C5: symbol CP -> zasilacz-v2-rescue:CP
- D1: symbol D_Schottky -> zasilacz-v2-rescue:D_Schottky
- J1: symbol USB_B -> zasilacz-v2-rescue:USB_B
- J2, J3, J4, J5, J6: symbol Conn_01x04 -> zasilacz-v2-rescue:Conn_01x04
- L1: symbol L -> zasilacz-v2-rescue:L
- R1, R2: symbol R -> zasilacz-v2-rescue:R
- U1: symbol MIC4576 -> zasilacz-v2-rescue:MIC4576
- U2: symbol TC7660H -> zasilacz-v2-rescue:TC7660H
