File: 2. HMI/PCB/HMI KiCad Project/HMI.sch (KiCad schematic (older format))
At the start: 71 parts, among them J1 Conn_01x05, J2 Conn_01x05, J3 Conn_01x04, J4 Conn_01x02, SW1 SW_DIP_x01, SW2 SW_DIP_x01, SW3 SW_DIP_x01, SW4 SW_DIP_x01, SW5 SW_DIP_x01, SW6 SW_DIP_x01, SW7 SW_DIP_x01, SW8 SW_DIP_x01, U1 PIC32MX130F064D-I/PT, U2 DOGL128-E, U3 74HC595

Commit message: Amiga rulez
Parts:
- C1, C10, C11, C12, C14, C15, C3, C4, C5, C6, C7, C8, C9: symbol C -> Device:C
- C13, C2: symbol CP -> Device:CP
- D1, D10, D11, D12, D13, D14, D15, D16, D17, D18, D19, D2, D20, D21, D22, D23, D24, D25, D26, D27, D28, D29, D3, D30, D31, D32, D4, D5, D6, D7, D8, D9: symbol D_Schottky -> Device:D_Schottky
- E1, E2, E3, E4, E5, E6, E7, E8: symbol Enkoder -> Różne-biblioteki-Artura:Enkoder
- J1, J2: symbol Conn_01x05 -> conn:Conn_01x05
- J3: symbol Conn_01x04 -> conn:Conn_01x04
- J4: symbol Conn_01x02 -> conn:Conn_01x02
- R1: symbol R -> Device:R
- SW1, SW2, SW3, SW4, SW5, SW6, SW7, SW8: symbol SW_DIP_x01 -> switches:SW_DIP_x01
- U1: symbol PIC32MX130F064D-I/PT -> HMI-rescue:PIC32MX130F064D-I_PT
- U2: symbol DOGL128-E -> Różne-biblioteki-Artura:DOGL128-E
- U3: symbol 74HC595 -> 74xx:74HC595
Connections:
- wire segments 313 -> 370
